File: tiramisu-dev-RP2354B/pcb/tiramisu-dev.kicad_pcb (KiCad board)
At the start: 4 copper layers, 154.1 x 147 mm, 324 parts, among them J1 TYPE-C-31-M-12, J2 SWD, SW1 TS-1187A-B-A-B, SW2 TS-1187A-B-A-B, U1 SRV05-4, U10 AMS1117-3.3, U100 HAL403SO, U101 HAL403SO, U102 HAL403SO, U103 HAL403SO, U104 HAL403SO, U105 HAL403SO, U106 HAL403SO, U107 HAL403SO, U108 HAL403SO, U109 HAL403SO, U11 RP2354B, U110 HAL403SO, U111 HAL403SO, U112 HAL403SO, U113 HAL403SO, U114 HAL403SO, U115 HAL403SO, U116 HAL403SO, U117 HAL403SO, U118 HAL403SO, U119 HAL403SO, U12 TLV73311PDBV, U120 HAL403SO, U121 HAL403SO, U122 HAL403SO, U123 HAL403SO, U124 HAL403SO, U125 HAL403SO, U126 HAL403SO, U127 HAL403SO, U128 HAL403SO, U129 HAL403SO, U13 HAL403SO, U130 HAL403SO, U131 HAL403SO, U132 HAL403SO, U14 HAL403SO, U15 HAL403SO, U16 HAL403SO, U17 HAL403SO, U18 HAL403SO, U19 HAL403SO, U2 CD74HC4067M, U20 HAL403SO, U21 HAL403SO, U22 HAL403SO, U23 HAL403SO, U24 HAL403SO, U25 HAL403SO, U26 HAL403SO, U27 HAL403SO, U28 HAL403SO, U29 HAL403SO, U3 CD74HC4067M, U30 HAL403SO, U31 HAL403SO, U32 HAL403SO, U33 HAL403SO, U34 HAL403SO, U35 HAL403SO, U36 HAL403SO, U37 HAL403SO, U38 HAL403SO, U39 HAL403SO, U4 CD74HC4067M, U40 HAL403SO, U41 HAL403SO, U42 HAL403SO, U43 HAL403SO, U44 HAL403SO, U45 HAL403SO, U46 HAL403SO, U47 HAL403SO, U48 HAL403SO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

Commit message: Update tiramisu-dev.kicad_pcb
Other:
- board text removed: "aim1k"
